File: Shelter.sch (KiCad schematic (older format))
At the start: 6 parts

Commit message: first commit
Parts:
- added J?: Conn_02x03_Top_Bottom, symbol Conn_02x03_Top_Bottom
Other:
- moved on the sheet: C?, Y?
Changed lines of the file:
@@
 L Crystal Y?
 U 1 1 5A43DC18
-P 5780 4004
-F 0 "Y?" H 5780 4154 50  0000 C CNN
-F 1 "Crystal" H 5780 3854 50  0000 C CNN
-F 2 "" H 5780 4004 50  0001 C CNN
-F 3 "" H 5780 4004 50  0001 C CNN
-	1    5780 4004
+P 5888 3794
+F 0 "Y?" H 5888 3944 50  0000 C CNN
+F 1 "Crystal" H 5888 3644 50  0000 C CNN
+F 2 "" H 5888 3794 50  0001 C CNN
+F 3 "" H 5888 3794 50  0001 C CNN
+	1    5888 3794
 	0    1    1    0
 $EndComp
@@
 L C C?
 U 1 1 5A43E12F
-P 6226 3850
-F 0 "C?" H 6251 3950 50  0000 L CNN
-F 1 "C" H 6251 3750 50  0000 L CNN
-F 2 "" H 6264 3700 50  0001 C CNN
-F 3 "" H 6226 3850 50  0001 C CNN
-	1    6226 3850
+P 6334 3640
+F 0 "C?" H 6359 3740 50  0000 L CNN
+F 1 "C" H 6359 3540 50  0000 L CNN
+F 2 "" H 6372 3490 50  0001 C CNN
+F 3 "" H 6334 3640 50  0001 C CNN
+	1    6334 3640
 	0    1    1    0
 $EndComp
@@
 L C C?
 U 1 1 5A43E2EE
-P 6224 4156
-F 0 "C?" H 6249 4256 50  0000 L CNN
-F 1 "C" H 6249 4056 50  0000 L CNN
-F 2 "" H 6262 4006 50  0001 C CNN
-F 3 "" H 6224 4156 50  0001 C CNN
-	1    6224 4156
+P 6332 3946
+F 0 "C?" H 6357 4046 50  0000 L CNN
+F 1 "C" H 6357 3846 50  0000 L CNN
+F 2 "" H 6370 3796 50  0001 C CNN
+F 3 "" H 6332 3946 50  0001 C CNN
+	1    6332 3946
 	0    1    1    0
 $EndComp
@@
 	1    0    0    -1
 $EndComp
+$Comp
+L Conn_02x03_Top_Bottom J?
+U 1 1 5A43EFC8
+P 8918 5428
+F 0 "J?" H 8968 5628 50  0000 C CNN
+F 1 "Conn_02x03_Top_Bottom" H 8968 5228 50  0000 C CNN
+F 2 "" H 8918 5428 50  0001 C CNN
+F 3 "" H 8918 5428 50  0001 C CNN
+	1    8918 5428
+	1    0    0    -1
+$EndComp
